File: pcb/iot-gateway.sch (EAGLE design)
At the start: 185 parts, among them CON1 6P-SH-TOP, CON2 6P-SH-TOP, CON3 2P-PH-TOP, J2 DCJACK-SMD, Q1 AO3401, Q2 AO3401, Q3 AO3400, Q4 AO3400, Q5 AO3400, T1 BC817, T3 BC817, T4 BC817, T5 BC817, U1 EFM32GG11B4XX_Q100, U10 CCS811, U11 MIC4682, U12 MIC4682, U13 MIC39101, U14 FS312F-G, U15 TP4056, U16 FS8205, U17 ER-TFT035-6, U2 SST26VF064B, U3 SST26VF016B, U4 ESP8266EX, U5 RFM69HW, U6 SIM800C, U7 SI7021, U8 SI7210, U9 BMP280, Y1 8 MHz, Y2 32.768 kHz, Y3 24 MHz

Commit message: Start schematic redesign
Parts:
- removed C10, C9: 1nF, Capacitor:CAPACITOR-0603
- removed C44, C45: 470pF, Capacitor:CAPACITOR-0603
- removed CON1: 6P-SH-TOP, JST:6P-SH-TOP
- removed D5: SK54L, Generic Diode:SK54L
- removed D6, D7: DSK24, Generic Diode:DSK24
- removed Q5: AO3400, Alpha Omega:AO3400
- removed R13: 100 Ohms, Resistor:RESISTOR-0603
- removed R56, R57: 100K Ohms, Resistor:RESISTOR-0603
- removed R65: 0 Ohms, Resistor:RESISTOR-0603
- removed T1, T3, T4: BC817, Generic BJT:BC817
- added C55, C60: 4.7uF, Capacitor:CAPACITOR-0603
- added C56, C61, C62, C69, C73: 100nF, Capacitor:CAPACITOR-0603
- added C57: 10uF, Capacitor:CAPACITOR-0603
- added C58, C59, C64, C65, C66, C67, C68: 470pF, Capacitor:CAPACITOR-0603
- added C63: 100uF, Capacitor:CAPACITOR-1206
- added D31: GREEN, LED:LED0603
- added D32: RED, LED:LED0603
- added L4: 1uH, Inductor:INDUCTOR-0805
- added L5: 470nH, Inductor:INDUCTOR-3.2XX2.5MM
- added L6: 4.7uH, Inductor:INDUCTOR-0603
- added R110: 510 Ohms, Resistor:RESISTOR-0603
- added R111: 330 Ohms, Resistor:RESISTOR-0603
- added R69, R70, R71, R72, R75, R76, R77, R78, R81, R82, R83, R84, R85, R86: 100K Ohms, Resistor:RESISTOR-0603
- added R73: 357K Ohms, Resistor:RESISTOR-0603
- added R74: 61.9K Ohms, Resistor:RESISTOR-0603
- added R79: 21K Ohms, Resistor:RESISTOR-0603
- added R80: 147K Ohms, Resistor:RESISTOR-0603
- added TC1: TC2050-IDC, TagConnect:TC2050-IDC
- added TP6, TP7, TP8: TESTPOINT-1.27MM, PADs:TESTPOINT-1.27MM
- added U18: EFM32GG11B820F2048GQ100, EFM32:EFM32GG11B820F2048GQ100
- added U21: 74LVC1G04, Logic:74LVC1G04
- C12, C22: value 10uF -> 100uF; device Capacitor:TANTALUM-CAPACITOR-CASE-A-EIA3216 -> Capacitor:CAPACITOR-1206
- C32: value 100nF -> 100uF; device Capacitor:CAPACITOR-0603 -> Capacitor:ALUMINIUM-CAPACITOR-CASE-D; OCLCSC (none) -> C97813; VOLTAGE (none) -> 25V
- C33: value 100nF -> 4.7uF
- C34: value 470uF -> 4.7uF; device Capacitor:ALUMINIUM-CAPACITOR-CASE-F -> Capacitor:CAPACITOR-0603; OCLCSC C294522 -> (none)
- C35, C41: value 470pF -> 1nF
- C36, C42, C51: value 10uF -> 100nF; device Capacitor:TANTALUM-CAPACITOR-CASE-A-EIA3216 -> Capacitor:CAPACITOR-0603
- C37: value 100nF -> 10nF
- C38: value 100nF -> 1uF
- C39: value 220uF -> 100uF; device Capacitor:ALUMINIUM-CAPACITOR-CASE-D -> Capacitor:CAPACITOR-1206; OCLCSC C189315 -> (none)
- C40: value 220uF -> 22uF; device Capacitor:ALUMINIUM-CAPACITOR-CASE-D -> Capacitor:CAPACITOR-1206; OCLCSC C189315 -> (none)
- C46: value 10uF -> 10pF; device Capacitor:TANTALUM-CAPACITOR-CASE-A-EIA3216 -> Capacitor:CAPACITOR-0603
- C47: value 100nF -> 100uF; device Capacitor:CAPACITOR-0603 -> Capacitor:CAPACITOR-1206
- C48: value 10uF -> 22uF; device Capacitor:TANTALUM-CAPACITOR-CASE-A-EIA3216 -> Capacitor:CAPACITOR-1206
- C49: value 100nF -> 10uF
- D2: value RED -> LED1206
- D3: value SMAJ12A -> LED1206; device TVS:SMAJ12A -> LED:LED1206
- D4: value SK54L -> SMAJ24A; device Generic Diode:SK54L -> TVS:SMAJ24A; OCLCSC C129816 -> (none)
- J2: value DCJACK-SMD -> DCJACK; device DC Jack:DCJACK-SMD -> DC Jack:DCJACK
- L2: value 68 uH -> 4.7uH; device Inductor:INDUCTOR-12X12X7MM -> Inductor:INDUCTOR-6X6MM; CURRENT (none) -> 3A; OCLCSC C182146 -> C326336
- L3: value 68 uH -> 2.2uH; device Inductor:INDUCTOR-12X12X7MM -> Inductor:INDUCTOR-5X5MM; CURRENT (none) -> 2.62A; OCLCSC C182146 -> C114791
- Q1, Q2: value AO3401 -> AO3400; device Alpha Omega:AO3401 -> Alpha Omega:AO3400
- R10: value 1 MOhms -> 22 Ohms
- R12: value 100 Ohms -> 10K Ohms
- R2: value 22 Ohms -> 330 Ohms
- R28: value 10K Ohms -> 330 Ohms
- R3: value 1K Ohms -> 22 Ohms
- R30: value 330 Ohms -> 22 Ohms
- R32, R67: value 10K Ohms -> 100K Ohms
- R39: value 10M Ohm -> 25m Ohms; device Resistor:RESISTOR-0603 -> Resistor:RESISTOR-1206; OCLCSC (none) -> C127700
- R40: value 10K Ohms -> 18.2K Ohms
- R42: value 10M Ohm -> 1M Ohms
- R43: value 10K Ohms -> 243K Ohms
- R44: value 3.01K Ohms -> 12m Ohms; device Resistor:RESISTOR-0603 -> Resistor:RESISTOR-1206; OCLCSC (none) -> C175759
- R45: value 953 Ohms -> 1.69M Ohms
- R46: value 300K Ohms -> 100K Ohms
- R47: value 47K Ohms -> 100K Ohms
- R48: value 3.01K Ohms -> 324K Ohms
- R49: value 1.2K Ohms -> 2K Ohms
- R50, R53: value 10K Ohms -> 100 Ohms
- R51, R54: value 100K Ohms -> 1 MOhms
- R52: value 100K Ohms -> 100 Ohms
- R55: value 47K Ohms -> 100 Ohms
- R58: value 1K Ohms -> 309K Ohms
- R59: value 100 Ohms -> 71.5K Ohms
- R61: value 100K Ohms -> 178K Ohms
- R62: value 1.5K Ohms -> 60.4K Ohms
- R63: value 10M Ohm -> 100K Ohms
- R9: value 1 MOhms -> 10K Ohms; MF (none) -> VISHAY
- TP1, TP2, TP3, TP4, TP5: value TESTPOINT -> TESTPOINT-1.27MM; device PADs:TESTPOINT -> PADs:TESTPOINT-1.27MM
- U$1: value GECKO -> GECKO-14MM; device Silkscreen:GECKO -> Silkscreen:GECKO-14MM
- U1: value EFM32GG11B4XX_Q100 -> 74LVC1G08; device EFM32:EFM32GG11B4XX_Q100 -> Logic:74LVC1G08
- U11: value MIC4682 -> LT4040; device Microchip:MIC4682 -> Analog Devices:LT4040
- U12: value MIC4682 -> LT8610; device Microchip:MIC4682 -> Analog Devices:LT8610
- U13: value MIC39101 -> LTC2942; device Microchip:MIC39101 -> Analog Devices:LTC2942
- U15: value TP4056 -> FS8205; device TP4056:TP4056 -> Fortune:FS8205
- U16: value FS8205 -> MIC23159; device Fortune:FS8205 -> Microchip:MIC23159
- U17: value ER-TFT035-6 -> ER-TFT035-6-BOT; device BuyDisplay:ER-TFT035-6 -> BuyDisplay:ER-TFT035-6-BOT
- Y1, Y3: device Crystal:CRYSTAL2-SMD-5X3 -> Crystal:CRYSTAL2-SMD-5032
Connections:
- net !WIFI_RST renamed !WIFI_RESET
- removed net !BAT_STDBY: R61.1, U1.PC6, U15.!STDBY
- removed net !TFT_IRQ: U1.PA13, U17.X-/!IRQ!
- removed net !VREG_ERR: R67.1, U1.PF11, U13.FLG
- removed net 4V2_SENSE: C41.C1, R51.1, R52.2, U1.PD5
- removed net 5V0_SENSE: C44.C1, R54.1, R55.2, U1.PD4
- removed net BTN_1: C9.C1, R12.2, R9.1, U1.PB1
- removed net BTN_2: C10.C1, R10.1, R13.2, U1.PB2
- removed net BTN_3: C11.C1, R11.1, R14.2, U1.PB3
- removed net N$32: Q5.G, R2.1
- removed net N$55: R12.1, S2.1, S2.2
- removed net N$56: R13.1, S3.1, S3.2
- removed net VBAT_SENSE: C45.C1, R56.1, R57.2, U1.PD6
- removed net VIN: C32.C1, C33.C1, C34.+, F1.1, R39.2, R42.2, R46.2, U11.IN, U12.IN
- removed net VIN_SENSE: C35.C1, R46.1, R47.2, U1.PD7
- new net !5V0_BACKUP: R72.1, U11.!PFO, U21.1.A
- new net !BAT_FAULT: R67.1, U11.!FAULT
- new net !TFT_TOUCH_IRQ: R47.1, U17.X-/!IRQ!
- new net !TFT_TOUCH_RESET: R46.1, U17.Y-/!RST!
- new net !UI_BTN1: C41.C1, R54.1, R55.2
- new net !UI_BTN2: C35.C1, R51.1, R52.2
- new net !UI_BTN3: C11.C1, R11.1, R14.2
- new net 12V0: C32.+, C33.C1, C36.C1, D4.C, F1.1, R80.2, U12.EN/UV, U12.VIN
- new net 12V0_UNFUSED: F1.2, J2.C
- new net 12V0_VSENSE: C64.C1, R79.2, R80.1
- new net 1V8: C34.C1, L6.1, U18.DVDD
- new net 3V3_FB: R58.1, R59.2, U16.FB@1
- new net 3V3_PGOOD: R60.1, U16.PG@1
- new net 4V2_EN: R76.2, U16.EN@0
- new net 4V2_FB: R73.1, R74.2, U16.FB@0
- new net 4V2_PGOOD: R75.1, U16.PG@0
- new net 4V2_VSENSE: C65.C1, R81.2, R82.1
- new net 5V0_FB: R45.1, R48.2, U11.BSTFB, U11.RSTFB
- new net 5V0_ISENSE: C68.C1, U11.CLPROG
- new net 5V0_NBU: Q1.S, R44.1, U11.CLN
- new net 5V0_NBU_NSENS: C39.C1, C40.C1, C42.C1, C46.C1, L2.2, R110.2, R42.2, R44.2, R61.2, U11.OVSNS, U11.VIN, U12.BIAS
- new net 5V0_NBU_NSENS_FB: C46.C2, R42.1, R43.2, U12.FB
- new net 5V0_NBU_NSENS_PGOOD: R77.1, U12.PG
- new net 5V0_NBU_NSENS_SYNC: R78.2, U12.SYNC
- new net 5V0_PGOOD: R71.1, U11.!RST
- new net 5V0_VSENSE: C66.C1, R83.2, R84.1
- new net N$12: R40.2, U12.RT
- new net N$13: C37.C1, U12.TR/SS
- new net N$14: C38.C1, U12.INTVCC
- new net N$15: C43.C1, L2.1, U12.SW
- new net N$58: TP7.TP, U6.UART2_TXD
- new net N$59: R55.1, S2.1, S2.2
- new net N$90: R111.2, U21.1.Y
- new net N$91: D31.A, R110.1
- new net N$92: D32.A, R111.1
- new net PF_THRESH: R61.1, R62.2, U11.PFI
- new net VBAT_NSENS: CON3-1.S, R39.1, U13.VBAT/SENSE-
- new net VBAT_VSENSE: C67.C1, R85.2, R86.1
- new net WIFI_LED: D3.A, U4.IO4
- net !BAT_CHRG: now also R63.1, U11.!CHRG; no longer R60.1, U1.PC7, U15.!CHRG
- net !CCS811_IRQ: no longer U1.PE9
- net !CCS811_RESET: no longer U1.PE11
- net !CCS811_WAKE: no longer U1.PE10
- net !GSM_DTR: no longer U1.PC5
- net !GSM_RING: no longer U1.PC4
- net !RESET: now also R69.1, TC1-10(!RESET!).S, U18.!RESET; no longer CON1-2.S, U1.!RESET
- net !TFT_RESET: now also R32.1; no longer U1.PA12, U17.Y-/!RST!
- net 3V3: now also C12.C1, C22.C1, C57.C1, C69.C1, C73.C1, L4.2, R32.2, R46.2, R47.2, R51.2, R54.2, R58.2, R63.2, R69.2, R71.2, R72.2, R75.2, R77.2, TC1-1(VTARGET).S, U1.PWR.GND, U16.SNS@1, U18.AVDD, U18.IOVDD0@0, U18.IOVDD0@1, U18.IOVDD0@2, U18.IOVDD0@3, U18.IOVDD0@4, U18.VREGVDD, U21.PWR.VCC; no longer C12.+, C46.+, C47.C1, C51.+, CON1-1.S, R10.2, R61.2, R9.2, U1.AVDD@0, U1.AVDD@1, U1.DVDD, U1.IOVDD0@0, U1.IOVDD0@1, U1.IOVDD0@2, U1.IOVDD0@3, U1.IOVDD0@4, U13.OUT
- net 4V2: now also C62.C1, C63.C1, L5.1, R73.2, R82.2, U16.SNS@0; no longer C22.+, C42.+, C43.C1, D2.A, D6.C, Q1.S, R51.2
- net 5V0: now also C47.C1, C48.C1, C55.C1, C56.C1, C60.C1, C61.C1, Q1.D, R45.2, R84.2, U11.F0, U11.F1, U11.F2, U11.VSYS, U16.AVIN@0, U16.AVIN@1, U16.EN@1, U16.VIN@0, U16.VIN@1; no longer C36.+, C38.C1, C40.+, C50.C1, D7.A, L2.2, Q2.G, R44.2, R53.2, R54.2, U15.CE, U15.VCC
- net GBAT: now also C51.C2, U13.GND, U15.S2; no longer C49.C2, R63.2, U16.S2
- net GND: now also C12.C2, C22.C2, C25.C2, C26.C2, C27.C2, C32.-, C34.C2, C36.C2, C39.C2, C40.C2, C42.C2, C48.C2, C49.C2, C55.C2, C56.C2, C57.C2, C58.C2, C59.C2, C60.C2, C61.C2, C62.C2, C63.C2, C64.C2, C65.C2, C66.C2, C67.C2, C68.C2, C69.C2, C73.C2, D31.C, D32.C, J2.O, Q2.S, R12.1, R2.1, R28.1, R31.1, R48.1, R59.1, R70.1, R74.1, R76.1, R78.1, R79.1, R81.1, R83.1, R85.1, R9.1, TC1-3(GND).S, U1.PWR.VCC, U11.BSTOFF, U11.CHGOFF, U11.GND, U11.NTC, U12.GND, U12.PGND, U15.S1, U16.AGND@0, U16.AGND@1, U16.PGND@0, U16.PGND@1, U16.PGND@2, U18.VREGVSS, U18.VSS@0, U18.VSS@1, U18.VSS@2, U18.VSS@3, U21.PWR.GND; no longer C10.C2, C12.-, C22.-, C25.C1, C26.C1, C27.C1, C32.C2, C34.-, C36.-, C39.-, C40.-, C42.-, C43.C2, C44.C2, C45.C2, C46.-, C48.-, C51.-, C9.C2, CON1-6.S, D3.A, D5.A, J2.2, Q5.S, R45.1, R47.1, R50.1, R52.1, R55.1, R57.1, R58.2, R63.1, T1.E, T3.E, U1.VSS@0, U1.VSS@1, U1.VSS@2, U1.VSS@3, U11.GND@1, U11.GND@2, U11.GND@3, U11.SHDN, U12.GND@1, U12.GND@2, U12.GND@3, U12.SHDN, U13.GND@0, U13.GND@1, U13.GND@2, U13.GND@3, U15.GND@0, U15.GND@1, U15.TEMP, U16.S1
- net GSM_LED_EN: now also U1.1.A; no longer R28.2, U1.PA10
- net GSM_PWRKEY: no longer U1.PA9
- net GSM_RF_SYNC: no longer U1.PA8
- net GSM_STATUS: no longer U1.PA7
- net I2C0_SCL_SENS: no longer U1.PE13
- net I2C0_SDA_SENS: no longer U1.PE12
- net I2C1_SCL_TFT: no longer U1.PB12
- net I2C1_SDA_TFT: no longer U1.PB11
- net LED_DI: now also R10.2; no longer R2.2, U1.PB0
- net MAG_ALERT: no longer U1.PE15
- net MAIN_HFXTAL_N: no longer U1.PB14
- net MAIN_HFXTAL_P: no longer U1.PB13
- net MAIN_LFXTAL_N: no longer U1.PB8
- net MAIN_LFXTAL_P: no longer U1.PB7
- net N$16: now also D2.C, R28.2; no longer R31.2, R32.2, T4.B
- net N$17: now also D2.A, U1.1.Y; no longer R30.2, T4.C
- net N$19: now also Q4.D; no longer Q5.D
- net N$23: now also TP8.TP, U6.VRTC; no longer R31.1, T3.C, T4.E
- net N$24: now also Q3.G, R30.2, R31.2; no longer D2.C, R30.1
- net N$29: now also D3.C, R2.2; no longer R28.1, T3.B
- net N$34: now also Q2.G, R9.2; no longer T1.B
- net N$35: now also Q2.D; no longer T1.C
- net N$36: now also C43.C2, U12.BST; no longer D4.C, L2.1, U11.SW
- net N$37: now also Q1.G, U11.IGATE; no longer R44.1, R45.2, U11.FB
- net N$38: now also L3.1, U11.SW; no longer R39.1, R40.2, U11.ISET
- net N$4: now also U1.1.B; no longer R32.1
- net N$40: now also R49.2, U11.PROG; no longer D5.C, L3.1, U12.SW
- net N$41: now also R50.1, U14.VCC; no longer R48.1, R49.2, U12.FB
- net N$42: now also R53.2, U14.CS; no longer R42.1, R43.2, U12.ISET
- net N$43: now also U14.OC, U15.G1; no longer C37.C1, C39.+, D6.A, L3.2, Q1.G, R48.2, R50.2
- net N$44: now also U14.OD, U15.G2; no longer D7.C, Q2.S, U13.EN, U13.IN
- net N$46: now also L4.1, U16.SW@1; no longer R62.2, U15.PROG
- net N$47: now also C58.C1, U16.SS@1; no longer U14.OC, U16.G1
- net N$48: now also C59.C1, U16.SS@0; no longer U14.OD, U16.G2
- net N$49: now also L5.2, U16.SW@0; no longer R59.1, U14.VCC
- net N$50: now also L6.2, U18.VREGSW; no longer R58.1, U14.CS
- net N$51: now also TP6.TP, U6.UART2_RXD; no longer D3.C, F1.2, J2.1
- net N$52: now also Q4.G, R10.1, R12.2; no longer Q4.D, R65.1
- net N$53: now also R52.1, S3.1, S3.2; no longer R65.2, U17.LEDK@1
- net N$54: now also U17.LEDK@1
- net N$9: now also U18.DECOUPLE; no longer U1.DECOUPLE
- net QSPI_CLK: now also U18.PF6; no longer U1.PF6
- net QSPI_CS0: now also U18.PF7; no longer U1.PF7
- net QSPI_D0: now also U18.PD9; no longer U1.PD9
- net QSPI_D1: now also U18.PD10; no longer U1.PD10
- net QSPI_D2: now also U18.PD11; no longer U1.PD11
- net QSPI_D3: now also U18.PD12; no longer U1.PD12
- net RFM_IRQ: now also R70.2; no longer U1.PA6
- net RFM_RESET: no longer U1.PA4
- net SIM_DATA: now also C27.C1; no longer C27.C2
- net SIM_VDD: now also C25.C1, C26.C1; no longer C25.C2, C26.C2
- net SWCLK: now also TC1-4(TCK/SWCLK).S, U18.PF0; no longer CON1-3.S, U1.PF0
- net SWDIO: now also TC1-2(TMS/SWDIO).S, U18.PF1; no longer CON1-4.S, U1.PF1
- net SWO: now also TC1-6(TDO/SWO).S, U18.PF2; no longer CON1-5.S, U1.PF2
- net TFT_DC: no longer U1.PA14
- net TIM3_CC2_BUZZ: no longer U1.PA15
- net US0_CLK_WIFI: no longer U1.PC9
- net US0_CS_WIFI: no longer U1.PC8
- net US0_MISO_WIFI: no longer U1.PC10
- net US0_MOSI_WIFI: no longer U1.PC11
- net US1_CLK_TFT: no longer U1.PD2
- net US1_CS_TFT: no longer U1.PD3
- net US1_MISO_TFT: no longer U1.PD1
- net US1_MOSI_TFT: no longer U1.PD0
- net US2_CTS_GSM: no longer U1.PC1
- net US2_RTS_GSM: no longer U1.PC0
- net US2_RX_GSM: no longer U1.PC3
- net US2_TX_GSM: no longer U1.PC2
- net US3_CLK_RFM: no longer U1.PA2
- net US3_CS_RFM: no longer U1.PA3
- net US3_MISO_RFM: no longer U1.PA1
- net US3_MOSI_RFM: no longer U1.PA0
- net VBAT: now also C50.C1, C51.C1, L3.2, R39.2, R50.2, R86.2, U11.BAT, U13.VDD/SENSE+; no longer C48.+, CON3-1.S, Q1.D, Q2.D, R56.2, R59.2, U15.BAT
- net VIN_DET: now also J2.DT; no longer J2.3, U1.PF12
- net WIFI_EN: no longer U1.PE4
- net WIFI_IRQ: no longer U1.PE3
- net WTIM2_CC1_TFT_BL: now also R30.1; no longer Q3.G, Q4.G, U1.PB10
Other:
- note removed: "4.2V Regulator"
- note removed: "5V & 3.3V Regulator"
- note removed: "BMP280 - Pressure and Temperature sensor"
- note removed: "Battery charger"
- note removed: "Battery connections"
- note removed: "Battery protection"
- note removed: "Battery voltage sense"
- note removed: "Buttons"
- note removed: "Buzzer"
- note removed: "CCS811 - Air Quality sensor"
- note removed: "Coef. = 100/200 = 0.5"
- note removed: "Coef. = 47/147 ~ 0.31973"
- note removed: "Coef. = 47/347 ~ 0.13545"
- note removed: "Debugger Connection"
- note removed: "Decouple"
- note removed: "High Frequency Crystal"
- note removed: "I2C Pull-ups"
- note removed: "Io(max) ~ 2A DS pag. 5"
- note removed: "LED"
- note removed: "LED Decouple"
- note removed: "Low Frequency Crystal"
- note removed: "Main power input"
- note removed: "Power rails sense"
- note removed: "SIM Card"
- note removed: "SPI Flash"
- note removed: "SPI Flash Decouple"
- note removed: "Si7021 - RH and Temperature sensor"
- note removed: "Si7210 - Hall effect and Temperature sensor"
- note removed: "Vo = 1.23 * (R3/R4 + 1) Vo ~ 4.31V"
- note removed: "Vo = 1.23 * (R3/R4 + 1) Vo ~ 5.11V"
