File: pcb/main/iot-gateway-main.sch (EAGLE design)
At the start: 261 parts, among them CON1 6P-SH-TOP, CON2 3P-SH-TOP, CON3 2P-PH-TOP, CON4 6P-SH-TOP, CON5 3P-SH-TOP, CON6 5P-SH-TOP, CON7 2P-PH-TOP, Q1 AO3400, Q2 AO3400, Q3 AO3400, Q4 FS8205, T1 BC817, U1 SST26VF064B, U10 SIM800C, U11 SI7021, U12 SI7210, U13 BMP280, U14 CCS811, U15 TMG39933, U16 ER-TFT035-6-BOT, U17 74LVC1G11, U18 74LVC1G17, U19 LTC4313-1, U2 EFM32GG11B820F2048GQ100, U20 LT8640S, U21 MIC23159, U22 74LVC1G04, U23 LTC2942, U24 LTC4040, U25 FS312F-G, U3 SST26VF016B, U4 ESP8266EX, U5 RFM69HW, U6 74LVC1G332, U7 74LVC1G332, U8 74LVC1G32, U9 74LVC1G08, X1 24 MHz, X2 32.768 kHz, X3 26 MHz

Commit message: Sync
Parts:
- R63: value 100K Ohms -> 10K Ohms
Changed lines of the file:
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@@
 <?xml version="1.0" encoding="utf-8"?>
 <!DOCTYPE eagle SYSTEM "eagle.dtd">
-<eagle version="9.5.2">
+<eagle version="9.6.1">
 <drawing>
 <settings>
@@
 <part name="3V391" library="Supply Symbol" deviceset="3V3" device=""/>
 <part name="3V381" library="Supply Symbol" deviceset="3V3" device=""/>
-<part name="R63" library="Resistor" deviceset="RESISTOR" device="-0603" value="100K Ohms"/>
+<part name="R63" library="Resistor" deviceset="RESISTOR" device="-0603" value="10K Ohms"/>
 <part name="D6" library="TVS" deviceset="SP0502BAJT" device=""/>
 <part name="GND113" library="Supply Symbol" deviceset="GND" device=""/>
@@
 <instance part="F1" gate="G$1" x="48.26" y="50.8" smashed="yes">
 <attribute name="OCLCSC" x="48.26" y="50.8" size="1.778" layer="96" display="off"/>
-<attribute name="HOLD" x="48.26" y="46.736" size="1.778" layer="97" align="top-left"/>
-<attribute name="TRIP" x="48.26" y="44.196" size="1.778" layer="97" align="top-left"/>
+<attribute name="HOLD" x="48.26" y="46.736" size="1.778" layer="97" align="top-left" display="both"/>
+<attribute name="TRIP" x="48.26" y="44.196" size="1.778" layer="97" align="top-left" display="both"/>
 <attribute name="NAME" x="48.26" y="55.6006" size="1.778" layer="95" ratio="10" rot="SR0"/>
 </instance>
