File: pcb/usb-pd/iot-gateway-usb-pd.sch (EAGLE design)
At the start: 39 parts, among them CON1 2P-PH-TOP, CON2 6P-SH-TOP, CON3 3P-SH-TOP, CON4 5P-SH-TOP, J1 DCJACK, Q1 AO3401, Q2 AO3401, U1 FUSB302MPX, U2 74LVC1G04, U3 74LVC1G08, U4 MIC2019, U5 LTC4412

Commit message: Sync
Changed lines of the file:
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@@
 <?xml version="1.0" encoding="utf-8"?>
 <!DOCTYPE eagle SYSTEM "eagle.dtd">
-<eagle version="9.5.2">
+<eagle version="9.6.1">
 <drawing>
 <settings>
@@
 <instance part="F2" gate="G$1" x="294.64" y="48.26" smashed="yes">
 <attribute name="OCLCSC" x="294.64" y="48.26" size="1.778" layer="96" display="off"/>
-<attribute name="HOLD" x="294.64" y="44.196" size="1.778" layer="97" align="top-left"/>
-<attribute name="TRIP" x="294.64" y="41.656" size="1.778" layer="97" align="top-left"/>
+<attribute name="HOLD" x="294.64" y="44.196" size="1.778" layer="97" align="top-left" display="both"/>
+<attribute name="TRIP" x="294.64" y="41.656" size="1.778" layer="97" align="top-left" display="both"/>
 <attribute name="NAME" x="294.64" y="53.0606" size="1.778" layer="95" ratio="10" rot="SR0"/>
 </instance>
@@
 <instance part="F1" gate="G$1" x="96.52" y="347.98" smashed="yes">
 <attribute name="OCLCSC" x="96.52" y="347.98" size="1.778" layer="96" display="off"/>
-<attribute name="HOLD" x="96.52" y="343.916" size="1.778" layer="97" align="top-left"/>
-<attribute name="TRIP" x="96.52" y="341.376" size="1.778" layer="97" align="top-left"/>
+<attribute name="HOLD" x="96.52" y="343.916" size="1.778" layer="97" align="top-left" display="both"/>
+<attribute name="TRIP" x="96.52" y="341.376" size="1.778" layer="97" align="top-left" display="both"/>
 <attribute name="NAME" x="96.52" y="352.7806" size="1.778" layer="95" ratio="10" rot="SR0"/>
 </instance>
